Commit message: Cambios del URDF

File: src/BRAZO_URDF_V3/urdf/BRAZO_URDF_V3.urdf (robot description, URDF)
Before this commit: robot BRAZO_URDF_V3, 7 links, 6 joints
Links:
- added link world
Joints:
- added joint base_joint: type fixed, parent world, child base_link, origin xyz=0.0 0.0 0.17 rpy=0 0 0
- joint GRIPPER DERECHO: mimic (none) -> joint=GRIPPER_IZQUIERDO multiplier=1 offset=0
