Commit message: Hice varios cambios y parece que funcionan hasta 3.9

File: brazo_urdf_nuevo/brazorobot_actualizado/urdf/brazorobot_actualizado.urdf (robot description, URDF)
Before this commit: robot brazorobot_actualizado.SLDASM, 8 links, 7 joints
Links:
- link link_1: geometry collision mesh filename=package://brazorobot_actualizado/meshes/link_1.STL; visual mesh filename=package://brazorobot_actualizado/meshes/link_1.STL
- link link_2: geometry collision mesh filename=package://brazorobot_actualizado/meshes/link_2.STL; visual mesh filename=package://brazorobot_actualizado/meshes/link_2.STL
- link link_3: geometry collision mesh filename=package://brazorobot_actualizado/meshes/link_3.STL; visual mesh filename=package://brazorobot_actualizado/meshes/link_3.STL
- link link_4: geometry collision mesh filename=package://brazorobot_actualizado/meshes/link_4.STL; visual mesh filename=package://brazorobot_actualizado/meshes/link_4.STL
- link link_5: geometry collision mesh filename=package://brazorobot_actualizado/meshes/link_5.STL; visual mesh filename=package://brazorobot_actualizado/meshes/link_5.STL
- link link_6: geometry collision mesh filename=package://brazorobot_actualizado/meshes/link_6.STL; visual mesh filename=package://brazorobot_actualizado/meshes/link_6.STL
- link link_7: geometry collision mesh filename=package://brazorobot_actualizado/meshes/link_7.STL; visual mesh filename=package://brazorobot_actualizado/meshes/link_7.STL

File: src/brazo_urdf_nuevo/brazorobot_actualizado/urdf/brazorobot_actualizado.urdf (robot description, URDF)
Before this commit: robot brazorobot_actualizado.SLDASM, 7 links, 6 joints
Links:
- link link_1: geometry collision mesh filename=package://brazorobot_actualizado/meshes/link_1.STL; visual mesh filename=package://brazorobot_actualizado/meshes/link_1.STL
- link link_2: geometry collision mesh filename=package://brazorobot_actualizado/meshes/link_2.STL; visual mesh filename=package://brazorobot_actualizado/meshes/link_2.STL
- link link_3: geometry collision mesh filename=package://brazorobot_actualizado/meshes/link_3.STL; visual mesh filename=package://brazorobot_actualizado/meshes/link_3.STL
- link link_4: geometry collision mesh filename=package://brazorobot_actualizado/meshes/link_4.STL; visual mesh filename=package://brazorobot_actualizado/meshes/link_4.STL
- link link_5: geometry collision mesh filename=package://brazorobot_actualizado/meshes/link_5.STL; visual mesh filename=package://brazorobot_actualizado/meshes/link_5.STL
- link link_6: geometry collision mesh filename=package://brazorobot_actualizado/meshes/link_6.STL; visual mesh filename=package://brazorobot_actualizado/meshes/link_6.STL
- link link_7: geometry collision mesh filename=package://brazorobot_actualizado/meshes/link_7.STL; visual mesh filename=package://brazorobot_actualizado/meshes/link_7.STL
